File: Button_LED.brd (EAGLE design)
At the start: 68.6 x 53.3 mm, 5 parts

Commit message: Fixed error with direction of LED in button LED circuit diagram
Connections:
- removed net N$6 (its old number): D2.A, R1.1, U1.GND.
- new net N$7: D2.K, R1.1, U1.GND.
- net N$5: now also D2.A; no longer D2.K
Changed lines of the file:
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@@
 <element value="" name="U1" library="AUTODESK_CIRCUITS_BREADBOARD" package="ARDUINO_UNO" x="5" y="10.08"></element><element value="" name="S1" library="AUTODESK_CIRCUITS_BREADBOARD" package="TL1105" x="5" y="22.78"></element><element value="1k‎Ω" name="R1" library="AUTODESK_CIRCUITS_BREADBOARD" package="0207/10" x="5" y="35.480000000000004"></element><element value="" name="D2" library="AUTODESK_CIRCUITS_BREADBOARD" package="LED5MM" x="5" y="48.18"></element><element value="1k‎Ω" name="R3" library="AUTODESK_CIRCUITS_BREADBOARD" package="0207/10" x="5" y="60.879999999999995"></element></elements>
 <signals>
-<signal name="N$1"><contactref element="S1" pad="2"></contactref></signal><signal name="N$2"><contactref element="S1" pad="1"></contactref></signal><signal name="N$3"><contactref element="S1" pad="3"></contactref><contactref element="R1" pad="2"></contactref><wire x1="2.75" y1="19.53" x2="10.08" y2="35.480000000000004" width="0" layer="19" extent="1-1"></wire><contactref element="U1" pad="8"></contactref><wire x1="10.08" y1="35.480000000000004" x2="46.656" y2="60.879999999999995" width="0" layer="19" extent="1-1"></wire></signal><signal name="N$4"><contactref element="U1" pad="5V"></contactref><contactref element="S1" pad="4"></contactref><wire x1="43.1" y1="12.620000000000001" x2="7.25" y2="19.53" width="0" layer="19" extent="1-1"></wire></signal><signal name="N$5"><contactref element="D2" pad="K"></contactref><contactref element="R3" pad="2"></contactref><wire x1="6.27" y1="48.18" x2="10.08" y2="60.879999999999995" width="0" layer="19" extent="1-1"></wire></signal><signal name="N$6"><contactref element="D2" pad="A"></contactref><contactref element="U1" pad="GND."></contactref><wire x1="3.73" y1="48.18" x2="48.18" y2="12.620000000000001" width="0" layer="19" extent="1-1"></wire><contactref element="R1" pad="1"></contactref><wire x1="48.18" y1="12.620000000000001" x2="-0.08000000000000007" y2="35.480000000000004" width="0" layer="19" extent="1-1"></wire></signal><signal name="N$7"><contactref element="R3" pad="1"></contactref><contactref element="U1" pad="7"></contactref><wire x1="-0.08000000000000007" y1="60.879999999999995" x2="50.72" y2="60.879999999999995" width="0" layer="19" extent="1-1"></wire></signal></signals>
+<signal name="N$1"><contactref element="S1" pad="2"></contactref></signal><signal name="N$2"><contactref element="S1" pad="1"></contactref></signal><signal name="N$3"><contactref element="S1" pad="3"></contactref><contactref element="R1" pad="2"></contactref><wire x1="2.75" y1="19.53" x2="10.08" y2="35.480000000000004" width="0" layer="19" extent="1-1"></wire><contactref element="U1" pad="8"></contactref><wire x1="10.08" y1="35.480000000000004" x2="46.656" y2="60.879999999999995" width="0" layer="19" extent="1-1"></wire></signal><signal name="N$4"><contactref element="U1" pad="5V"></contactref><contactref element="S1" pad="4"></contactref><wire x1="43.1" y1="12.620000000000001" x2="7.25" y2="19.53" width="0" layer="19" extent="1-1"></wire></signal><signal name="N$5"><contactref element="R3" pad="2"></contactref><contactref element="D2" pad="A"></contactref><wire x1="10.08" y1="60.879999999999995" x2="3.73" y2="48.18" width="0" layer="19" extent="1-1"></wire></signal><signal name="N$6"><contactref element="R3" pad="1"></contactref><contactref element="U1" pad="7"></contactref><wire x1="-0.08000000000000007" y1="60.879999999999995" x2="50.72" y2="60.879999999999995" width="0" layer="19" extent="1-1"></wire></signal><signal name="N$7"><contactref element="D2" pad="K"></contactref><contactref element="U1" pad="GND."></contactref><wire x1="6.27" y1="48.18" x2="48.18" y2="12.620000000000001" width="0" layer="19" extent="1-1"></wire><contactref element="R1" pad="1"></contactref><wire x1="48.18" y1="12.620000000000001" x2="-0.08000000000000007" y2="35.480000000000004" width="0" layer="19" extent="1-1"></wire></signal></signals>
 </board>
 </drawing>
